File: SequencerMidiController/BassStation_Sequencer_MidiInterface.kicad_pcb (KiCad board)
At the start: 2 copper layers, 194 parts, among them J1 MIDI IN, J2 MIDI OUT, J4 Conn_02x10_Odd_Even, J5 Barrel_Jack_Switch, J6 Conn_02x02_Counter_Clockwise, J7 Conn_02x05_Odd_Even, J8 Conn_01x07, Q1 HX2301A, SW1 Rotary_Encoder_Switch, SW2 SW_DIP_x04, SW3 SW_SPST, SW4 SW_SPDT-2MS1T1B1M2QES, SW5 SW_SPST, SW6 SW_DIP_x04, SW7 SW_SPST, U1 PCB-SPST_RGB-LED-Counter-Cloc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, U10 PCB-SPST_RGB-LED-Counter-Cloc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, U11 PCB-SPST_RGB-LED-Counter-Cloc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, U12 PCB-SPST_RGB-LED-Counter-Cloc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, U13 PCB-SPST_RGB-LED-Counter-Cloc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, U14 PCB-SPST_RGB-LED-Counter-Cloc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, U15 PCB-SPST_RGB-LED-Counter-Cloc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, U16 PCB-SPST_RGB-LED-Counter-Cloc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, U17 PCB-SPST_RGB-LED-Counter-Cloc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, U18 PCB-SPST_RGB-LED-Counter-Cloc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, U19 PCB-SPST_RGB-LED-Counter-Cloc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, U2 PCB-SPST_RGB-LED-Counter-Cloc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, U20 PCB-SPST_RGB-LED-Counter-Cloc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, U21 PCB-SPST_RGB-LED-Counter-Cloc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, U22 PCB-SPST_RGB-LED-Counter-Cloc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, U23 PCB-SPST_RGB-LED-Counter-Cloc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, U24 PCB-SPST_RGB-LED-Counter-Cloc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, U25 PCB-SPST_RGB-LED-Counter-Cloc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, U26 PCB-SPST_RGB-LED-Counter-Cloc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, U27 PCB-SPST_RGB-LED-Counter-Cloc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, U28 PCB-SPST_RGB-LED-Counter-Cloc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, U29 PCB-SPST_RGB-LED-Counter-Cloc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, U3 PCB-SPST_RGB-LED-Counter-Cloc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, U30 PCB-SPST_RGB-LED-Counter-Cloc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, U31 PCB-SPST_RGB-LED-Counter-Cloc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, U32 PCB-SPST_RGB-LED-Counter-Cloc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, U33 STM32G0B1_KxTxN_LQFP32, U34 ADG2188, U35 ADP5587-ACPZ_LFCSP24, U36 TLC5955DCA_HTSSOP56, U37 TLC5955DCA_HTSSOP56, U38 TPS563200, U39 TPS563200, U4 PCB-SPST_RGB-LED-Counter-Cloc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, U40 SE8233X2, U41 MCP1703A-3302_SOT223, U42 74LVC1G34, U43 6N135S, U5 PCB-SPST_RGB-LED-Counter-Cloc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, U6 PCB-SPST_RGB-LED-Counter-Cloc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, U7 PCB-SPST_RGB-LED-Counter-Cloc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, U8 PCB-SPST_RGB-LED-Counter-Cloc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, U9 PCB-SPST_RGB-LED-Counter-Cloc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

Commit message: RevA Layout draft completed
- Needs tidy up
- Add test points
Parts:
- removed J6: Conn_02x02_Counter_Clockwise, Connector_PinHeader_2.54mm:PinHeader_2x02_P2.54mm_Vertical
- removed R13, R15, R16, R17, R31: 220R, Resistor_SMD:R_0805_2012Metric_Pad1.20x1.40mm_HandSolder
- removed the REF** at (315.3, 190.1)
- removed the REF** at (285.3, 190.1)
- removed the REF** at (255.3, 190.1)
- removed the REF** at (225.2, 190.1)
- removed the REF** at (195.3, 190.1)
- removed SW6: SW_DIP_x04, Button_Switch_THT:SW_DIP_SPSTx04_Slide_9.78x12.34mm_W7.62mm_P2.54mm
- removed TP10, TP11, TP12, TP13, TP14, TP15, TP16, TP17, TP18, TP19, TP20, TP21, TP22, TP23, TP24, TP25, TP26, TP27, TP28, TP29, TP30, TP31, TP32, TP33, TP34, TP35, TP36, TP37, TP38, TP39, TP40, TP41, TP42, TP43, TP44, TP45, TP46, TP47, TP48, TP49: TestPoint, TestPoint:TestPoint_Pad_D1.0mm
- added JP1: Jumper_NC_Small, Jumper:SolderJumper-2_P1.3mm_Bridged_RoundedPad1.0x1.5mm, B.Cu at (121.8, 128.0)
- added JP2: Jumper_NC_Small, Jumper:SolderJumper-2_P1.3mm_Bridged_RoundedPad1.0x1.5mm, B.Cu at (118.9, 128.0)
- added JP3: Jumper_NC_Small, Jumper:SolderJumper-2_P1.3mm_Bridged_RoundedPad1.0x1.5mm, B.Cu at (115.8, 128.0)
- added REF**: Adafruit_1611_NPTH, PCB_SW_LED:Adafruit_1611_NPTH, F.Cu at (312.1, 183.9)
- added REF**: Adafruit_1611_NPTH, PCB_SW_LED:Adafruit_1611_NPTH, F.Cu at (282.1, 183.9)
- added REF**: Adafruit_1611_NPTH, PCB_SW_LED:Adafruit_1611_NPTH, F.Cu at (252.1, 183.9)
- added REF**: Adafruit_1611_NPTH, PCB_SW_LED:Adafruit_1611_NPTH, F.Cu at (222.1, 183.9)
- added REF**: Adafruit_1611_NPTH, PCB_SW_LED:Adafruit_1611_NPTH, F.Cu at (192.1, 183.9)
- C10, C20, C21, C22, C23, C9, D2, R11, R12, R22, R23, R24, U34, U35, U36, U37: moved to B.Cu
- J4: footprint Connector_PinHeader_2.54mm:PinHeader_2x10_P2.54mm_Vertical -> Connector_IDC:IDC-Header_2x10_P2.54mm_Horizontal
- R20: value 100R -> 220R
- SW2: value SW_DIP_x04 -> SW_SPDT-2MS1T1B1M2QES; footprint Button_Switch_THT:SW_DIP_SPSTx04_Slide_9.78x12.34mm_W7.62mm_P2.54mm -> DailywellSwitches:Dailywell_SPDT
- SW4: value SW_SPDT-2MS1T1B1M2QES -> SW_DIP_x04; footprint DailywellSwitches:Dailywell_SPDT -> Button_Switch_THT:SW_DIP_SPSTx04_Slide_9.78x12.34mm_W7.62mm_P2.54mm
- SW5, SW7: footprint Button_Switch_THT:SW_TH_Tactile_Omron_B3F-10xx -> Button_Switch_THT:SW_PUSH-12mm
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Connections:
- R11 pad 2: Net-(J6-Pad4) -> /MCU/SWDCLK
- R12 pad 1: Net-(J6-Pad3) -> /MCU/SWDCLK
- R20 pad 1: GND -> /Input Keyscan and RGB LED Driver/ADP5587_WRITE
- R20 pad 2: Net-(R20-Pad2) -> +3V3
- R30 pad 1: /Input Keyscan and RGB LED Driver/ADP5587_WRITE -> Net-(R30-Pad1)
- SW2 pad 1: /CrossPoint Output Switching/A0 -> GND
- SW2 pad 2: /CrossPoint Output Switching/A1 -> /Input Keyscan and RGB LED Driver/ADP5587_WRITEPROTECT
- SW2 pad 3: /CrossPoint Output Switching/A2 -> Net-(R30-Pad1)
- SW4 pad 1: GND -> /Input Keyscan and RGB LED Driver/DIPSW1
- SW4 pad 2: /Input Keyscan and RGB LED Driver/ADP5587_WRITEPROTECT -> /Input Keyscan and RGB LED Driver/DIPSW2
- SW4 pad 3: Net-(R31-Pad1) -> /Input Keyscan and RGB LED Driver/DIPSW3
- U1 pad 1: /Input Keyscan and RGB LED Driver/OUTB1 -> /Input Keyscan and RGB LED Driver/LEDBK1
- U1 pad 2: /Input Keyscan and RGB LED Driver/OUTG1 -> /Input Keyscan and RGB LED Driver/LEDGK1
- U1 pad 3: /Input Keyscan and RGB LED Driver/OUTR1 -> /Input Keyscan and RGB LED Driver/LEDRK1
- U1 pad 4: +3V3 -> /PSU/+5V_RGB
- U1 pad 5: +3V3 -> /PSU/+5V_RGB
- U1 pad 6: +3V3 -> /PSU/+5V_RGB
- U10 pad 1: /Input Keyscan and RGB LED Driver/OUTB10 -> /Input Keyscan and RGB LED Driver/LEDBK10
- U10 pad 2: /Input Keyscan and RGB LED Driver/OUTG10 -> /Input Keyscan and RGB LED Driver/LEDGK10
- U10 pad 3: /Input Keyscan and RGB LED Driver/OUTR10 -> /Input Keyscan and RGB LED Driver/LEDRK10
- U10 pad 4: +3V3 -> /PSU/+5V_RGB
- U10 pad 5: +3V3 -> /PSU/+5V_RGB
- U10 pad 6: +3V3 -> /PSU/+5V_RGB
- U11 pad 1: /Input Keyscan and RGB LED Driver/OUTB11 -> /Input Keyscan and RGB LED Driver/LEDBK11
- U11 pad 2: /Input Keyscan and RGB LED Driver/OUTG11 -> /Input Keyscan and RGB LED Driver/LEDGK11
- U11 pad 3: /Input Keyscan and RGB LED Driver/OUTR11 -> /Input Keyscan and RGB LED Driver/LEDRK11
- U11 pad 4: +3V3 -> /PSU/+5V_RGB
- U11 pad 5: +3V3 -> /PSU/+5V_RGB
- U11 pad 6: +3V3 -> /PSU/+5V_RGB
- U12 pad 1: /Input Keyscan and RGB LED Driver/OUTB12 -> /Input Keyscan and RGB LED Driver/LEDBK12
- U12 pad 2: /Input Keyscan and RGB LED Driver/OUTG12 -> /Input Keyscan and RGB LED Driver/LEDGK12
- U12 pad 3: /Input Keyscan and RGB LED Driver/OUTR12 -> /Input Keyscan and RGB LED Driver/LEDRK12
- U12 pad 4: +3V3 -> /PSU/+5V_RGB
- U12 pad 5: +3V3 -> /PSU/+5V_RGB
- U12 pad 6: +3V3 -> /PSU/+5V_RGB
- U13 pad 1: /Input Keyscan and RGB LED Driver/OUTB13 -> /Input Keyscan and RGB LED Driver/LEDBK13
- U13 pad 2: /Input Keyscan and RGB LED Driver/OUTG13 -> /Input Keyscan and RGB LED Driver/LEDGK13
- U13 pad 3: /Input Keyscan and RGB LED Driver/OUTR13 -> /Input Keyscan and RGB LED Driver/LEDRK13
- U13 pad 4: +3V3 -> /PSU/+5V_RGB
- U13 pad 5: +3V3 -> /PSU/+5V_RGB
- U13 pad 6: +3V3 -> /PSU/+5V_RGB
- U14 pad 1: /Input Keyscan and RGB LED Driver/OUTB14 -> /Input Keyscan and RGB LED Driver/LEDBK14
- U14 pad 2: /Input Keyscan and RGB LED Driver/OUTG14 -> /Input Keyscan and RGB LED Driver/LEDGK14
- U14 pad 3: /Input Keyscan and RGB LED Driver/OUTR14 -> /Input Keyscan and RGB LED Driver/LEDRK14
- U14 pad 4: +3V3 -> /PSU/+5V_RGB
- U14 pad 5: +3V3 -> /PSU/+5V_RGB
- U14 pad 6: +3V3 -> /PSU/+5V_RGB
- U15 pad 1: /Input Keyscan and RGB LED Driver/OUTB15 -> /Input Keyscan and RGB LED Driver/LEDBK15
- U15 pad 2: /Input Keyscan and RGB LED Driver/OUTG15 -> /Input Keyscan and RGB LED Driver/LEDGK15
- U15 pad 3: /Input Keyscan and RGB LED Driver/OUTR15 -> /Input Keyscan and RGB LED Driver/LEDRK15
- U15 pad 4: +3V3 -> /PSU/+5V_RGB
- U15 pad 5: +3V3 -> /PSU/+5V_RGB
- U15 pad 6: +3V3 -> /PSU/+5V_RGB
- U16 pad 1: /Input Keyscan and RGB LED Driver/OUTB16 -> /Input Keyscan and RGB LED Driver/LEDBK16
- U16 pad 2: /Input Keyscan and RGB LED Driver/OUTG16 -> /Input Keyscan and RGB LED Driver/LEDGK16
- U16 pad 3: /Input Keyscan and RGB LED Driver/OUTR16 -> /Input Keyscan and RGB LED Driver/LEDRK16
- U16 pad 4: +3V3 -> /PSU/+5V_RGB
- U16 pad 5: +3V3 -> /PSU/+5V_RGB
- U16 pad 6: +3V3 -> /PSU/+5V_RGB
- U17 pad 1: /Input Keyscan and RGB LED Driver/OUTB17 -> /Input Keyscan and RGB LED Driver/LEDBK17
- U17 pad 2: /Input Keyscan and RGB LED Driver/OUTG17 -> /Input Keyscan and RGB LED Driver/LEDGK17
- U17 pad 3: /Input Keyscan and RGB LED Driver/OUTR17 -> /Input Keyscan and RGB LED Driver/LEDRK17
- U17 pad 4: +3V3 -> /PSU/+5V_RGB
- U17 pad 5: +3V3 -> /PSU/+5V_RGB
- U17 pad 6: +3V3 -> /PSU/+5V_RGB
- U18 pad 1: /Input Keyscan and RGB LED Driver/OUTB18 -> /Input Keyscan and RGB LED Driver/LEDBK18
- U18 pad 2: /Input Keyscan and RGB LED Driver/OUTG18 -> /Input Keyscan and RGB LED Driver/LEDGK18
- U18 pad 3: /Input Keyscan and RGB LED Driver/OUTR18 -> /Input Keyscan and RGB LED Driver/LEDRK18
- U18 pad 4: +3V3 -> /PSU/+5V_RGB
- U18 pad 5: +3V3 -> /PSU/+5V_RGB
- U18 pad 6: +3V3 -> /PSU/+5V_RGB
- U19 pad 1: /Input Keyscan and RGB LED Driver/OUTB19 -> /Input Keyscan and RGB LED Driver/LEDBK19
- U19 pad 2: /Input Keyscan and RGB LED Driver/OUTG19 -> /Input Keyscan and RGB LED Driver/LEDGK19
- U19 pad 3: /Input Keyscan and RGB LED Driver/OUTR19 -> /Input Keyscan and RGB LED Driver/LEDRK19
- U19 pad 4: +3V3 -> /PSU/+5V_RGB
- U19 pad 5: +3V3 -> /PSU/+5V_RGB
- U19 pad 6: +3V3 -> /PSU/+5V_RGB
- U2 pad 1: /Input Keyscan and RGB LED Driver/OUTB2 -> /Input Keyscan and RGB LED Driver/LEDBK2
- U2 pad 2: /Input Keyscan and RGB LED Driver/OUTG2 -> /Input Keyscan and RGB LED Driver/LEDGK2
- U2 pad 3: /Input Keyscan and RGB LED Driver/OUTR2 -> /Input Keyscan and RGB LED Driver/LEDRK2
- U2 pad 4: +3V3 -> /PSU/+5V_RGB
- U2 pad 5: +3V3 -> /PSU/+5V_RGB
- U2 pad 6: +3V3 -> /PSU/+5V_RGB
- U20 pad 1: /Input Keyscan and RGB LED Driver/OUTB20 -> /Input Keyscan and RGB LED Driver/LEDBK20
- U20 pad 2: /Input Keyscan and RGB LED Driver/OUTG20 -> /Input Keyscan and RGB LED Driver/LEDGK20
- U20 pad 3: /Input Keyscan and RGB LED Driver/OUTR20 -> /Input Keyscan and RGB LED Driver/LEDRK20
- U20 pad 4: +3V3 -> /PSU/+5V_RGB
- U20 pad 5: +3V3 -> /PSU/+5V_RGB
- U20 pad 6: +3V3 -> /PSU/+5V_RGB
- U21 pad 1: /Input Keyscan and RGB LED Driver/OUTB21 -> /Input Keyscan and RGB LED Driver/LEDBK21
- U21 pad 2: /Input Keyscan and RGB LED Driver/OUTG21 -> /Input Keyscan and RGB LED Driver/LEDGK21
- U21 pad 3: /Input Keyscan and RGB LED Driver/OUTR21 -> /Input Keyscan and RGB LED Driver/LEDRK21
- U21 pad 4: +3V3 -> /PSU/+5V_RGB
- U21 pad 5: +3V3 -> /PSU/+5V_RGB
- U21 pad 6: +3V3 -> /PSU/+5V_RGB
- U22 pad 1: /Input Keyscan and RGB LED Driver/OUTB22 -> /Input Keyscan and RGB LED Driver/LEDBK22
- U22 pad 2: /Input Keyscan and RGB LED Driver/OUTG22 -> /Input Keyscan and RGB LED Driver/LEDGK22
- U22 pad 3: /Input Keyscan and RGB LED Driver/OUTR22 -> /Input Keyscan and RGB LED Driver/LEDRK22
- U22 pad 4: +3V3 -> /PSU/+5V_RGB
- U22 pad 5: +3V3 -> /PSU/+5V_RGB
- U22 pad 6: +3V3 -> /PSU/+5V_RGB
- U23 pad 1: /Input Keyscan and RGB LED Driver/OUTB23 -> /Input Keyscan and RGB LED Driver/LEDBK23
- U23 pad 2: /Input Keyscan and RGB LED Driver/OUTG23 -> /Input Keyscan and RGB LED Driver/LEDGK23
- U23 pad 3: /Input Keyscan and RGB LED Driver/OUTR23 -> /Input Keyscan and RGB LED Driver/LEDRK23
- U23 pad 4: +3V3 -> /PSU/+5V_RGB
- U23 pad 5: +3V3 -> /PSU/+5V_RGB
- U23 pad 6: +3V3 -> /PSU/+5V_RGB
- U24 pad 1: /Input Keyscan and RGB LED Driver/OUTB24 -> /Input Keyscan and RGB LED Driver/LEDBK24
- U24 pad 2: /Input Keyscan and RGB LED Driver/OUTG24 -> /Input Keyscan and RGB LED Driver/LEDGK24
- U24 pad 3: /Input Keyscan and RGB LED Driver/OUTR24 -> /Input Keyscan and RGB LED Driver/LEDRK24
- U24 pad 4: +3V3 -> /PSU/+5V_RGB
- U24 pad 5: +3V3 -> /PSU/+5V_RGB
- U24 pad 6: +3V3 -> /PSU/+5V_RGB
- U25 pad 1: /Input Keyscan and RGB LED Driver/OUTB25 -> /Input Keyscan and RGB LED Driver/LEDBK25
- U25 pad 2: /Input Keyscan and RGB LED Driver/OUTG25 -> /Input Keyscan and RGB LED Driver/LEDGK25
- U25 pad 3: /Input Keyscan and RGB LED Driver/OUTR25 -> /Input Keyscan and RGB LED Driver/LEDRK25
- U25 pad 4: +3V3 -> /PSU/+5V_RGB
- U25 pad 5: +3V3 -> /PSU/+5V_RGB
- U25 pad 6: +3V3 -> /PSU/+5V_RGB
- U26 pad 1: /Input Keyscan and RGB LED Driver/OUTB26 -> /Input Keyscan and RGB LED Driver/LEDBK26
- U26 pad 2: /Input Keyscan and RGB LED Driver/OUTG26 -> /Input Keyscan and RGB LED Driver/LEDGK26
- U26 pad 3: /Input Keyscan and RGB LED Driver/OUTR26 -> /Input Keyscan and RGB LED Driver/LEDRK26
- U26 pad 4: +3V3 -> /PSU/+5V_RGB
- U26 pad 5: +3V3 -> /PSU/+5V_RGB
- U26 pad 6: +3V3 -> /PSU/+5V_RGB
- U27 pad 1: /Input Keyscan and RGB LED Driver/OUTB27 -> /Input Keyscan and RGB LED Driver/LEDBK27
- U27 pad 2: /Input Keyscan and RGB LED Driver/OUTG27 -> /Input Keyscan and RGB LED Driver/LEDGK27
- U27 pad 3: /Input Keyscan and RGB LED Driver/OUTR27 -> /Input Keyscan and RGB LED Driver/LEDRK27
- U27 pad 4: +3V3 -> /PSU/+5V_RGB
- U27 pad 5: +3V3 -> /PSU/+5V_RGB
- U27 pad 6: +3V3 -> /PSU/+5V_RGB
- U28 pad 1: /Input Keyscan and RGB LED Driver/OUTB28 -> /Input Keyscan and RGB LED Driver/LEDBK28
- U28 pad 2: /Input Keyscan and RGB LED Driver/OUTG28 -> /Input Keyscan and RGB LED Driver/LEDGK28
- U28 pad 3: /Input Keyscan and RGB LED Driver/OUTR28 -> /Input Keyscan and RGB LED Driver/LEDRK28
- U28 pad 4: +3V3 -> /PSU/+5V_RGB
- U28 pad 5: +3V3 -> /PSU/+5V_RGB
- U28 pad 6: +3V3 -> /PSU/+5V_RGB
- U29 pad 1: /Input Keyscan and RGB LED Driver/OUTB29 -> /Input Keyscan and RGB LED Driver/LEDBK29
- U29 pad 2: /Input Keyscan and RGB LED Driver/OUTG29 -> /Input Keyscan and RGB LED Driver/LEDGK29
- U29 pad 3: /Input Keyscan and RGB LED Driver/OUTR29 -> /Input Keyscan and RGB LED Driver/LEDRK29
- U29 pad 4: +3V3 -> /PSU/+5V_RGB
- U29 pad 5: +3V3 -> /PSU/+5V_RGB
- U29 pad 6: +3V3 -> /PSU/+5V_RGB
- U3 pad 1: /Input Keyscan and RGB LED Driver/OUTB3 -> /Input Keyscan and RGB LED Driver/LEDBK3
- U3 pad 2: /Input Keyscan and RGB LED Driver/OUTG3 -> /Input Keyscan and RGB LED Driver/LEDGK3
- U3 pad 3: /Input Keyscan and RGB LED Driver/OUTR3 -> /Input Keyscan and RGB LED Driver/LEDRK3
- U3 pad 4: +3V3 -> /PSU/+5V_RGB
- U3 pad 5: +3V3 -> /PSU/+5V_RGB
- U3 pad 6: +3V3 -> /PSU/+5V_RGB
- U30 pad 1: /Input Keyscan and RGB LED Driver/OUTB30 -> /Input Keyscan and RGB LED Driver/LEDBK30
- U30 pad 2: /Input Keyscan and RGB LED Driver/OUTG30 -> /Input Keyscan and RGB LED Driver/LEDGK30
- U30 pad 3: /Input Keyscan and RGB LED Driver/OUTR30 -> /Input Keyscan and RGB LED Driver/LEDRK30
- U30 pad 4: +3V3 -> /PSU/+5V_RGB
- U30 pad 5: +3V3 -> /PSU/+5V_RGB
- U30 pad 6: +3V3 -> /PSU/+5V_RGB
- U31 pad 1: /Input Keyscan and RGB LED Driver/OUTB31 -> /Input Keyscan and RGB LED Driver/LEDBK31
- U31 pad 2: /Input Keyscan and RGB LED Driver/OUTG31 -> /Input Keyscan and RGB LED Driver/LEDGK31
- U31 pad 3: /Input Keyscan and RGB LED Driver/OUTR31 -> /Input Keyscan and RGB LED Driver/LEDRK31
- U31 pad 4: +3V3 -> /PSU/+5V_RGB
- U31 pad 5: +3V3 -> /PSU/+5V_RGB
- U31 pad 6: +3V3 -> /PSU/+5V_RGB
- U32 pad 1: /Input Keyscan and RGB LED Driver/OUTB32 -> /Input Keyscan and RGB LED Driver/LEDBK32
- U32 pad 2: /Input Keyscan and RGB LED Driver/OUTG32 -> /Input Keyscan and RGB LED Driver/LEDGK32
- U32 pad 3: /Input Keyscan and RGB LED Driver/OUTR32 -> /Input Keyscan and RGB LED Driver/LEDRK32
- U32 pad 4: +3V3 -> /PSU/+5V_RGB
- U32 pad 5: +3V3 -> /PSU/+5V_RGB
- U32 pad 6: +3V3 -> /PSU/+5V_RGB
- U33 pad 1: /OLED_Display/DATA_COMMAND -> /MCU/SPI2_LAT
- U33 pad 10: /MCU/SPI1_GSCLK -> /OLED_Display/RESET
- U33 pad 12: Net-(U33-Pad12) -> /Input Keyscan and RGB LED Driver/ADP5587_INT
- U33 pad 2: /OLED_Display/RESET -> /MCU/SPI2_GSCLK
- U33 pad 21: /Input Keyscan and RGB LED Driver/ADP5587_INT -> Net-(U33-Pad21)
- U33 pad 31: /OLED_Display/DATA -> /MCU/SPI2_MOSI
- U33 pad 32: /OLED_Display/CLK -> /MCU/SPI2_CLK
- U33 pad 7: /MCU/SPI1_GSCLK -> /OLED_Display/DATA_COMMAND
- U33 pad 8: /MCU/SPI1_SCK -> /OLED_Display/CLK
- U33 pad 9: /MCU/SPI1_MOSI -> /OLED_Display/DATA
- U36 pad 1: /MCU/SPI1_MOSI -> /MCU/SPI2_MOSI
- U36 pad 10: /Input Keyscan and RGB LED Driver/OUTB6 -> /Input Keyscan and RGB LED Driver/LEDBK11
- U36 pad 11: /Input Keyscan and RGB LED Driver/OUTR6 -> /Input Keyscan and RGB LED Driver/LEDRK11
- U36 pad 12: /Input Keyscan and RGB LED Driver/OUTG6 -> /Input Keyscan and RGB LED Driver/LEDGK11
- U36 pad 13: /Input Keyscan and RGB LED Driver/OUTB2 -> /Input Keyscan and RGB LED Driver/LEDBK12
- U36 pad 14: /Input Keyscan and RGB LED Driver/OUTR2 -> /Input Keyscan and RGB LED Driver/LEDRK12
- U36 pad 15: /Input Keyscan and RGB LED Driver/OUTG2 -> /Input Keyscan and RGB LED Driver/LEDGK12
- U36 pad 16: /Input Keyscan and RGB LED Driver/OUTB3 -> /Input Keyscan and RGB LED Driver/LEDBK13
- U36 pad 17: /Input Keyscan and RGB LED Driver/OUTR3 -> /Input Keyscan and RGB LED Driver/LEDRK13
- U36 pad 18: /Input Keyscan and RGB LED Driver/OUTG3 -> /Input Keyscan and RGB LED Driver/LEDGK13
- U36 pad 19: /Input Keyscan and RGB LED Driver/OUTB7 -> /Input Keyscan and RGB LED Driver/LEDBK14
- U36 pad 2: /MCU/SPI1_SCK -> /MCU/SPI2_CLK
- U36 pad 20: /Input Keyscan and RGB LED Driver/OUTR7 -> /Input Keyscan and RGB LED Driver/LEDRK14
- U36 pad 21: /Input Keyscan and RGB LED Driver/OUTG7 -> /Input Keyscan and RGB LED Driver/LEDGK14
- U36 pad 22: /Input Keyscan and RGB LED Driver/OUTB4 -> /Input Keyscan and RGB LED Driver/LEDBK15
- U36 pad 23: /Input Keyscan and RGB LED Driver/OUTR4 -> /Input Keyscan and RGB LED Driver/LEDRK15
- U36 pad 24: /Input Keyscan and RGB LED Driver/OUTG4 -> /Input Keyscan and RGB LED Driver/LEDGK15
- U36 pad 25: /Input Keyscan and RGB LED Driver/OUTB8 -> /Input Keyscan and RGB LED Driver/LEDBK16
- U36 pad 26: /Input Keyscan and RGB LED Driver/OUTR8 -> /Input Keyscan and RGB LED Driver/LEDRK16
- U36 pad 27: /Input Keyscan and RGB LED Driver/OUTG8 -> /Input Keyscan and RGB LED Driver/LEDGK16
- U36 pad 3: /MCU/SPI1_GSCLK -> /MCU/SPI2_LAT
- U36 pad 30: /Input Keyscan and RGB LED Driver/OUTG12 -> /Input Keyscan and RGB LED Driver/LEDGK1
- U36 pad 31: /Input Keyscan and RGB LED Driver/OUTR12 -> /Input Keyscan and RGB LED Driver/LEDRK1
- U36 pad 32: /Input Keyscan and RGB LED Driver/OUTB12 -> /Input Keyscan and RGB LED Driver/LEDBK1
- U36 pad 33: /Input Keyscan and RGB LED Driver/OUTG16 -> /Input Keyscan and RGB LED Driver/LEDGK2
- U36 pad 34: /Input Keyscan and RGB LED Driver/OUTR16 -> /Input Keyscan and RGB LED Driver/LEDRK2
- U36 pad 35: /Input Keyscan and RGB LED Driver/OUTB16 -> /Input Keyscan and RGB LED Driver/LEDBK2
- U36 pad 36: /Input Keyscan and RGB LED Driver/OUTG11 -> /Input Keyscan and RGB LED Driver/LEDGK3
- U36 pad 37: /Input Keyscan and RGB LED Driver/OUTR11 -> /Input Keyscan and RGB LED Driver/LEDRK3
- U36 pad 38: /Input Keyscan and RGB LED Driver/OUTB11 -> /Input Keyscan and RGB LED Driver/LEDBK3
- U36 pad 39: /Input Keyscan and RGB LED Driver/OUTG15 -> /Input Keyscan and RGB LED Driver/LEDGK4
- U36 pad 4: /Input Keyscan and RGB LED Driver/OUTB5 -> /Input Keyscan and RGB LED Driver/LEDBK9
- U36 pad 40: /Input Keyscan and RGB LED Driver/OUTR15 -> /Input Keyscan and RGB LED Driver/LEDRK4
- U36 pad 41: /Input Keyscan and RGB LED Driver/OUTB15 -> /Input Keyscan and RGB LED Driver/LEDBK4
- U36 pad 42: /Input Keyscan and RGB LED Driver/OUTG14 -> /Input Keyscan and RGB LED Driver/LEDGK5
- U36 pad 43: /Input Keyscan and RGB LED Driver/OUTR14 -> /Input Keyscan and RGB LED Driver/LEDRK5
- U36 pad 44: /Input Keyscan and RGB LED Driver/OUTB14 -> /Input Keyscan and RGB LED Driver/LEDBK5
- U36 pad 45: /Input Keyscan and RGB LED Driver/OUTG10 -> /Input Keyscan and RGB LED Driver/LEDGK6
- U36 pad 46: /Input Keyscan and RGB LED Driver/OUTR10 -> /Input Keyscan and RGB LED Driver/LEDRK6
- U36 pad 47: /Input Keyscan and RGB LED Driver/OUTB10 -> /Input Keyscan and RGB LED Driver/LEDBK6
- U36 pad 48: /Input Keyscan and RGB LED Driver/OUTG13 -> /Input Keyscan and RGB LED Driver/LEDGK7
- U36 pad 49: /Input Keyscan and RGB LED Driver/OUTR13 -> /Input Keyscan and RGB LED Driver/LEDRK7
- U36 pad 5: /Input Keyscan and RGB LED Driver/OUTR5 -> /Input Keyscan and RGB LED Driver/LEDRK9
- U36 pad 50: /Input Keyscan and RGB LED Driver/OUTB13 -> /Input Keyscan and RGB LED Driver/LEDBK7
- U36 pad 51: /Input Keyscan and RGB LED Driver/OUTG9 -> /Input Keyscan and RGB LED Driver/LEDGK8
- U36 pad 52: /Input Keyscan and RGB LED Driver/OUTR9 -> /Input Keyscan and RGB LED Driver/LEDRK8
- U36 pad 53: /Input Keyscan and RGB LED Driver/OUTB9 -> /Input Keyscan and RGB LED Driver/LEDBK8
- U36 pad 55: /MCU/SPI1_GSCLK -> /MCU/SPI2_GSCLK
- U36 pad 6: /Input Keyscan and RGB LED Driver/OUTG5 -> /Input Keyscan and RGB LED Driver/LEDGK9
- U36 pad 7: /Input Keyscan and RGB LED Driver/OUTB1 -> /Input Keyscan and RGB LED Driver/LEDBK10
- U36 pad 8: /Input Keyscan and RGB LED Driver/OUTR1 -> /Input Keyscan and RGB LED Driver/LEDRK10
- U36 pad 9: /Input Keyscan and RGB LED Driver/OUTG1 -> /Input Keyscan and RGB LED Driver/LEDGK10
- U37 pad 10: /Input Keyscan and RGB LED Driver/OUTB22 -> /Input Keyscan and RGB LED Driver/LEDBK30
- U37 pad 11: /Input Keyscan and RGB LED Driver/OUTR22 -> /Input Keyscan and RGB LED Driver/LEDRK30
- U37 pad 12: /Input Keyscan and RGB LED Driver/OUTG22 -> /Input Keyscan and RGB LED Driver/LEDGK30
- U37 pad 13: /Input Keyscan and RGB LED Driver/OUTB18 -> /Input Keyscan and RGB LED Driver/LEDBK29
- U37 pad 14: /Input Keyscan and RGB LED Driver/OUTR18 -> /Input Keyscan and RGB LED Driver/LEDRK29
- U37 pad 15: /Input Keyscan and RGB LED Driver/OUTG18 -> /Input Keyscan and RGB LED Driver/LEDGK29
- U37 pad 16: /Input Keyscan and RGB LED Driver/OUTB19 -> /Input Keyscan and RGB LED Driver/LEDBK28
- U37 pad 17: /Input Keyscan and RGB LED Driver/OUTR19 -> /Input Keyscan and RGB LED Driver/LEDRK28
- U37 pad 18: /Input Keyscan and RGB LED Driver/OUTG19 -> /Input Keyscan and RGB LED Driver/LEDGK28
- U37 pad 19: /Input Keyscan and RGB LED Driver/OUTB23 -> /Input Keyscan and RGB LED Driver/LEDBK27
- U37 pad 2: /MCU/SPI1_SCK -> /MCU/SPI2_CLK
- U37 pad 20: /Input Keyscan and RGB LED Driver/OUTR23 -> /Input Keyscan and RGB LED Driver/LEDRK27
- U37 pad 21: /Input Keyscan and RGB LED Driver/OUTG23 -> /Input Keyscan and RGB LED Driver/LEDGK27
- U37 pad 22: /Input Keyscan and RGB LED Driver/OUTB20 -> /Input Keyscan and RGB LED Driver/LEDBK26
- U37 pad 23: /Input Keyscan and RGB LED Driver/OUTR20 -> /Input Keyscan and RGB LED Driver/LEDRK26
- U37 pad 24: /Input Keyscan and RGB LED Driver/OUTG20 -> /Input Keyscan and RGB LED Driver/LEDGK26
- U37 pad 25: /Input Keyscan and RGB LED Driver/OUTB24 -> /Input Keyscan and RGB LED Driver/LEDBK25
- U37 pad 26: /Input Keyscan and RGB LED Driver/OUTR24 -> /Input Keyscan and RGB LED Driver/LEDRK25
- U37 pad 27: /Input Keyscan and RGB LED Driver/OUTG24 -> /Input Keyscan and RGB LED Driver/LEDGK25
- U37 pad 3: /MCU/SPI1_GSCLK -> /MCU/SPI2_LAT
- U37 pad 30: /Input Keyscan and RGB LED Driver/OUTG28 -> /Input Keyscan and RGB LED Driver/LEDGK24
- U37 pad 31: /Input Keyscan and RGB LED Driver/OUTR28 -> /Input Keyscan and RGB LED Driver/LEDRK24
- U37 pad 32: /Input Keyscan and RGB LED Driver/OUTB28 -> /Input Keyscan and RGB LED Driver/LEDBK24
- U37 pad 33: /Input Keyscan and RGB LED Driver/OUTG32 -> /Input Keyscan and RGB LED Driver/LEDGK23
- U37 pad 34: /Input Keyscan and RGB LED Driver/OUTR32 -> /Input Keyscan and RGB LED Driver/LEDRK23
- U37 pad 35: /Input Keyscan and RGB LED Driver/OUTB32 -> /Input Keyscan and RGB LED Driver/LEDBK23
- U37 pad 36: /Input Keyscan and RGB LED Driver/OUTG27 -> /Input Keyscan and RGB LED Driver/LEDGK22
- U37 pad 37: /Input Keyscan and RGB LED Driver/OUTR27 -> /Input Keyscan and RGB LED Driver/LEDRK22
- U37 pad 38: /Input Keyscan and RGB LED Driver/OUTB27 -> /Input Keyscan and RGB LED Driver/LEDBK22
- U37 pad 39: /Input Keyscan and RGB LED Driver/OUTG31 -> /Input Keyscan and RGB LED Driver/LEDGK21
- U37 pad 4: /Input Keyscan and RGB LED Driver/OUTB21 -> /Input Keyscan and RGB LED Driver/LEDBK32
- U37 pad 40: /Input Keyscan and RGB LED Driver/OUTR31 -> /Input Keyscan and RGB LED Driver/LEDRK21
- U37 pad 41: /Input Keyscan and RGB LED Driver/OUTB31 -> /Input Keyscan and RGB LED Driver/LEDBK21
- U37 pad 42: /Input Keyscan and RGB LED Driver/OUTG30 -> /Input Keyscan and RGB LED Driver/LEDGK20
- U37 pad 43: /Input Keyscan and RGB LED Driver/OUTR30 -> /Input Keyscan and RGB LED Driver/LEDRK20
- U37 pad 44: /Input Keyscan and RGB LED Driver/OUTB30 -> /Input Keyscan and RGB LED Driver/LEDBK20
- U37 pad 45: /Input Keyscan and RGB LED Driver/OUTG26 -> /Input Keyscan and RGB LED Driver/LEDGK19
- U37 pad 46: /Input Keyscan and RGB LED Driver/OUTR26 -> /Input Keyscan and RGB LED Driver/LEDRK19
- U37 pad 47: /Input Keyscan and RGB LED Driver/OUTB26 -> /Input Keyscan and RGB LED Driver/LEDBK19
- U37 pad 48: /Input Keyscan and RGB LED Driver/OUTG29 -> /Input Keyscan and RGB LED Driver/LEDGK18
- U37 pad 49: /Input Keyscan and RGB LED Driver/OUTR29 -> /Input Keyscan and RGB LED Driver/LEDRK18
- U37 pad 5: /Input Keyscan and RGB LED Driver/OUTR21 -> /Input Keyscan and RGB LED Driver/LEDRK32
- U37 pad 50: /Input Keyscan and RGB LED Driver/OUTB29 -> /Input Keyscan and RGB LED Driver/LEDBK18
- U37 pad 51: /Input Keyscan and RGB LED Driver/OUTG25 -> /Input Keyscan and RGB LED Driver/LEDGK17
- U37 pad 52: /Input Keyscan and RGB LED Driver/OUTR25 -> /Input Keyscan and RGB LED Driver/LEDRK17
- U37 pad 53: /Input Keyscan and RGB LED Driver/OUTB25 -> /Input Keyscan and RGB LED Driver/LEDBK17
- U37 pad 55: /MCU/SPI1_GSCLK -> /MCU/SPI2_GSCLK
- U37 pad 6: /Input Keyscan and RGB LED Driver/OUTG21 -> /Input Keyscan and RGB LED Driver/LEDGK32
- U37 pad 7: /Input Keyscan and RGB LED Driver/OUTB17 -> /Input Keyscan and RGB LED Driver/LEDBK31
- U37 pad 8: /Input Keyscan and RGB LED Driver/OUTR17 -> /Input Keyscan and RGB LED Driver/LEDRK31
- U37 pad 9: /Input Keyscan and RGB LED Driver/OUTG17 -> /Input Keyscan and RGB LED Driver/LEDGK31
- U4 pad 1: /Input Keyscan and RGB LED Driver/OUTB4 -> /Input Keyscan and RGB LED Driver/LEDBK4
- U4 pad 2: /Input Keyscan and RGB LED Driver/OUTG4 -> /Input Keyscan and RGB LED Driver/LEDGK4
- U4 pad 3: /Input Keyscan and RGB LED Driver/OUTR4 -> /Input Keyscan and RGB LED Driver/LEDRK4
- U4 pad 4: +3V3 -> /PSU/+5V_RGB
- U4 pad 5: +3V3 -> /PSU/+5V_RGB
- U4 pad 6: +3V3 -> /PSU/+5V_RGB
- U5 pad 1: /Input Keyscan and RGB LED Driver/OUTB5 -> /Input Keyscan and RGB LED Driver/LEDBK5
- U5 pad 2: /Input Keyscan and RGB LED Driver/OUTG5 -> /Input Keyscan and RGB LED Driver/LEDGK5
- U5 pad 3: /Input Keyscan and RGB LED Driver/OUTR5 -> /Input Keyscan and RGB LED Driver/LEDRK5
- U5 pad 4: +3V3 -> /PSU/+5V_RGB
- U5 pad 5: +3V3 -> /PSU/+5V_RGB
- U5 pad 6: +3V3 -> /PSU/+5V_RGB
- U6 pad 1: /Input Keyscan and RGB LED Driver/OUTB6 -> /Input Keyscan and RGB LED Driver/LEDBK6
- U6 pad 2: /Input Keyscan and RGB LED Driver/OUTG6 -> /Input Keyscan and RGB LED Driver/LEDGK6
- U6 pad 3: /Input Keyscan and RGB LED Driver/OUTR6 -> /Input Keyscan and RGB LED Driver/LEDRK6
- U6 pad 4: +3V3 -> /PSU/+5V_RGB
- U6 pad 5: +3V3 -> /PSU/+5V_RGB
- U6 pad 6: +3V3 -> /PSU/+5V_RGB
- U7 pad 1: /Input Keyscan and RGB LED Driver/OUTB7 -> /Input Keyscan and RGB LED Driver/LEDBK7
- U7 pad 2: /Input Keyscan and RGB LED Driver/OUTG7 -> /Input Keyscan and RGB LED Driver/LEDGK7
- U7 pad 3: /Input Keyscan and RGB LED Driver/OUTR7 -> /Input Keyscan and RGB LED Driver/LEDRK7
- U7 pad 4: +3V3 -> /PSU/+5V_RGB
- U7 pad 5: +3V3 -> /PSU/+5V_RGB
- U7 pad 6: +3V3 -> /PSU/+5V_RGB
- U8 pad 1: /Input Keyscan and RGB LED Driver/OUTB8 -> /Input Keyscan and RGB LED Driver/LEDBK8
- U8 pad 2: /Input Keyscan and RGB LED Driver/OUTG8 -> /Input Keyscan and RGB LED Driver/LEDGK8
- U8 pad 3: /Input Keyscan and RGB LED Driver/OUTR8 -> /Input Keyscan and RGB LED Driver/LEDRK8
- U8 pad 4: +3V3 -> /PSU/+5V_RGB
- U8 pad 5: +3V3 -> /PSU/+5V_RGB
- U8 pad 6: +3V3 -> /PSU/+5V_RGB
- U9 pad 1: /Input Keyscan and RGB LED Driver/OUTB9 -> /Input Keyscan and RGB LED Driver/LEDBK9
- U9 pad 2: /Input Keyscan and RGB LED Driver/OUTG9 -> /Input Keyscan and RGB LED Driver/LEDGK9
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Routing:
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- added copper zone on F.Cu, net +5V
- added copper zone on F.Cu, net /PSU/+5V_RGB
- added copper zone on In1.Cu_5VRGB, net /PSU/+5V_RGB
- added copper zone on B.Cu, net GND
- added copper zone on F.Cu, net GND
- added copper zone on In2.Cu_GND, net GND
Other:
- board outline added: 251.5 x 99.1 mm
- copper layers 2 -> 4
- net class Default: clearance 0.2 -> 0.127; trace_width 0.25 -> 0.127; via_dia 0.8 -> 0.6; via_drill 0.4 -> 0.3
- rule trace_clearance: 0.2 -> 0.127
- rule trace_min: 0.2 -> 0.127
- rule via_min_drill: 0.3 -> 0.2

Commit message: Added mounting holes to corners of layout
Parts:
- added REF**: MountingHole_3.2mm_M3_Pad_Via, MountingHole:MountingHole_3.2mm_M3_Pad_Via, F.Cu at (86.4, 100.3)
- added REF**: MountingHole_3.2mm_M3_Pad_Via, MountingHole:MountingHole_3.2mm_M3_Pad_Via, F.Cu at (64.8, 100.3)
- added REF**: MountingHole_3.2mm_M3_Pad_Via, MountingHole:MountingHole_3.2mm_M3_Pad_Via, F.Cu at (86.4, 189.2)
- added REF**: MountingHole_3.2mm_M3_Pad_Via, MountingHole:MountingHole_3.2mm_M3_Pad_Via, F.Cu at (326.4, 189.2)
- added REF**: MountingHole_3.2mm_M3_Pad_Via, MountingHole:MountingHole_3.2mm_M3_Pad_Via, F.Cu at (326.4, 100.3)
- moved U42 11.5 mm to (180.8, 115.8), turned to 0 degrees
- moved J4 6.98 mm to (113.7, 108.5)
- moved R2 6.10 mm to (186.7, 115.8), turned to 90 degrees
- moved J2 5.08 mm to (181.6, 102.9)
- moved TP51 5.08 mm to (189.7, 115.8)
- moved D1 5.08 mm to (91.8, 121.4)
- moved J5 5.08 mm to (98.4, 109.2)
- moved Q1 5.08 mm to (95.9, 121.4)
- moved R5 5.08 mm to (94.5, 114.2)
- moved SW3 5.08 mm to (99.8, 113.9)
- moved TP3 5.08 mm to (99.8, 120.5)
- moved D2 5.08 mm to (161.3, 120.0)
- moved J1 5.08 mm to (154.9, 102.9)
- moved TP50 4.99 mm to (175.5, 115.8), turned to 270 degrees
- moved TP1 4.95 mm to (146.6, 116.2)
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Routing:
- net /CrossPoint Output Switching/X5: track 12.8 -> 22.9 mm
- net /CrossPoint Output Switching/X4: track 12.8 -> 22.7 mm
- net /CrossPoint Output Switching/X3: track 12.8 -> 22.1 mm
- net Net-(D2-Pad2): track 9.58 -> 18.4 mm, vias 1 -> 0
- net /CrossPoint Output Switching/Y4: track 8.46 -> 16.7 mm
- net /CrossPoint Output Switching/Y7: track 14.7 -> 22.5 mm
- net /CrossPoint Output Switching/Y6: track 12.8 -> 20.0 mm
- net /CrossPoint Output Switching/X7: track 15.3 -> 22.5 mm
- net +5V: track 300.0 -> 292.8 mm
- net /CrossPoint Output Switching/Y5: track 11.1 -> 18.0 mm
- net /CrossPoint Output Switching/X6: track 12.8 -> 19.6 mm
- net /CrossPoint Output Switching/X2: track 14.5 -> 21.2 mm
- net /CrossPoint Output Switching/Y3: track 7.61 -> 14.1 mm
- net Net-(R2-Pad1): track 10.5 -> 4.51 mm
- net +3V3: track 329.5 -> 335.4 mm
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Other:
- board size 251.5 x 99.1 mm -> 250.2 x 99.1 mm

Commit message: Completed RevA layout
Parts:
- removed the REF** at (192.1, 183.9)
- removed the REF** at (64.8, 100.3)
- removed the REF** at (86.4, 189.2)
- removed the REF** at (326.4, 189.2)
- removed the REF** at (312.1, 183.9)
- removed the REF** at (282.1, 183.9)
- removed the REF** at (252.1, 183.9)
- removed the REF** at (222.1, 183.9)
- added REF**: MountingHole_3.2mm_M3_Pad_Via, MountingHole:MountingHole_3.2mm_M3_Pad_Via, F.Cu at (206.2, 150.1)
- added REF**: Adafruit_1611_NPTH, PCB_SW_LED:Adafruit_1611_NPTH, F.Cu at (250.8, 196.6)
- added REF**: Adafruit_1611_NPTH, PCB_SW_LED:Adafruit_1611_NPTH, F.Cu at (220.8, 196.6)
- added REF**: Adafruit_1611_NPTH, PCB_SW_LED:Adafruit_1611_NPTH, F.Cu at (190.8, 196.6)
- added REF**: MountingHole_3.2mm_M3_Pad_Via, MountingHole:MountingHole_3.2mm_M3_Pad_Via, F.Cu at (205.7, 212.7)
- added REF**: MountingHole_3.2mm_M3_Pad_Via, MountingHole:MountingHole_3.2mm_M3_Pad_Via, F.Cu at (205.7, 100.3)
- added REF**: MountingHole_3.2mm_M3_Pad_Via, MountingHole:MountingHole_3.2mm_M3_Pad_Via, F.Cu at (86.4, 212.7)
- added REF**: MountingHole_3.2mm_M3_Pad_Via, MountingHole:MountingHole_3.2mm_M3_Pad_Via, F.Cu at (325.8, 212.7)
- added REF**: Adafruit_1611_NPTH, PCB_SW_LED:Adafruit_1611_NPTH, F.Cu at (310.8, 196.6)
- added REF**: Adafruit_1611_NPTH, PCB_SW_LED:Adafruit_1611_NPTH, F.Cu at (280.8, 196.6)
- added TP10: TestPoint, TestPoint:TestPoint_Pad_D1.0mm, F.Cu at (159.6, 152.1)
- added TP11: TestPoint, TestPoint:TestPoint_Pad_D1.0mm, F.Cu at (163.7, 148.0)
- added TP13: TestPoint, TestPoint:TestPoint_Pad_D1.0mm, F.Cu at (156.2, 149.4)
- added TP15: TestPoint, TestPoint:TestPoint_Pad_D1.0mm, F.Cu at (161.0, 147.8)
- added TP16: TestPoint, TestPoint:TestPoint_Pad_D1.0mm, F.Cu at (213.5, 212.5)
- added TP17: TestPoint, TestPoint:TestPoint_Pad_D1.0mm, F.Cu at (98.3, 201.4)
- added TP18: TestPoint, TestPoint:TestPoint_Pad_D1.0mm, F.Cu at (313.6, 159.9)
- added TP19: TestPoint, TestPoint:TestPoint_Pad_D1.0mm, F.Cu at (98.4, 166.9)
- added TP20: TestPoint, TestPoint:TestPoint_Pad_D1.0mm, F.Cu at (306.6, 159.9)
- added TP21: TestPoint, TestPoint:TestPoint_Pad_D1.0mm, F.Cu at (178.7, 135.9)
- added TP22: TestPoint, TestPoint:TestPoint_Pad_D1.0mm, F.Cu at (179.1, 138.9)
- added TP23: TestPoint, TestPoint:TestPoint_Pad_D1.0mm, F.Cu at (175.3, 140.6)
- added TP24: TestPoint, TestPoint:TestPoint_Pad_D1.0mm, F.Cu at (213.4, 160.5)
- added TP25: TestPoint, TestPoint:TestPoint_Pad_D1.0mm, F.Cu at (221.1, 160.0)
- added TP26: TestPoint, TestPoint:TestPoint_Pad_D1.0mm, F.Cu at (234.4, 160.0)
- added TP27: TestPoint, TestPoint:TestPoint_Pad_D1.0mm, F.Cu at (251.0, 160.0)
- added TP28: TestPoint, TestPoint:TestPoint_Pad_D1.0mm, F.Cu at (262.6, 160.0)
- added TP29: TestPoint, TestPoint:TestPoint_Pad_D1.0mm, F.Cu at (274.3, 159.9)
- added TP30: TestPoint, TestPoint:TestPoint_Pad_D1.0mm, F.Cu at (285.1, 159.9)
- added TP31: TestPoint, TestPoint:TestPoint_Pad_D1.0mm, F.Cu at (297.1, 159.9)
- added TP32: TestPoint, TestPoint:TestPoint_Pad_D1.0mm, F.Cu at (110.5, 132.1)
- added TP33: TestPoint, TestPoint:TestPoint_Pad_D1.0mm, F.Cu at (110.5, 129.5)
- added TP34: TestPoint, TestPoint:TestPoint_Pad_D1.0mm, F.Cu at (110.5, 127.0)
- added TP35: TestPoint, TestPoint:TestPoint_Pad_D1.0mm, F.Cu at (110.5, 124.5)
- added TP36: TestPoint, TestPoint:TestPoint_Pad_D1.0mm, F.Cu at (110.5, 121.9)
- added TP37: TestPoint, TestPoint:TestPoint_Pad_D1.0mm, F.Cu at (110.5, 119.4)
- added TP38: TestPoint, TestPoint:TestPoint_Pad_D1.0mm, F.Cu at (110.5, 116.8)
- added TP39: TestPoint, TestPoint:TestPoint_Pad_D1.0mm, F.Cu at (110.5, 114.3)
- added TP40: TestPoint, TestPoint:TestPoint_Pad_D1.0mm, F.Cu at (137.5, 122.6)
- added TP41: TestPoint, TestPoint:TestPoint_Pad_D1.0mm, F.Cu at (136.5, 112.9)
- added TP42: TestPoint, TestPoint:TestPoint_Pad_D1.0mm, F.Cu at (136.1, 125.2)
- added TP43: TestPoint, TestPoint:TestPoint_Pad_D1.0mm, F.Cu at (134.0, 112.9)
- added TP44: TestPoint, TestPoint:TestPoint_Pad_D1.0mm, F.Cu at (131.4, 112.9)
- added TP45: TestPoint, TestPoint:TestPoint_Pad_D1.0mm, F.Cu at (128.9, 112.9)
- added TP46: TestPoint, TestPoint:TestPoint_Pad_D1.0mm, F.Cu at (126.4, 112.9)
- added TP47: TestPoint, TestPoint:TestPoint_Pad_D1.0mm, F.Cu at (123.8, 112.9)
- added TP48: TestPoint, TestPoint:TestPoint_Pad_D1.0mm, F.Cu at (121.3, 112.9)
- added Y0: TestPoint, TestPoint:TestPoint_Pad_D1.0mm, F.Cu at (118.7, 112.9)
- D1: value BZT52C5V1 -> MMSZ4694T1G
- Q1: value HX2301A -> Si2323DS
- R5: value 100K -> 100R
- SW3: footprint Connector_Molex:Molex_KK-254_AE-6410-02A_1x02_P2.54mm_Vertical -> DailywellSwitches:Dailywell_SPDT
- moved TP5 118.5 mm to (108.0, 156.2), turned to 180 degrees
- moved D3 111.9 mm to (103.9, 153.5)
- moved R7 111.9 mm to (99.3, 158.0)
- moved C1 111.9 mm to (91.7, 150.7)
- moved C2 111.9 mm to (91.7, 148.2)
- moved C3 111.9 mm to (95.5, 156.8)
- moved C4 111.9 mm to (100.3, 150.7)
- moved C5 111.9 mm to (100.3, 148.2)
- moved L1 111.9 mm to (95.5, 141.9)
- moved R6 111.9 mm to (104.1, 156.2)
- moved U38 111.9 mm to (91.7, 156.8)
- moved R8 111.9 mm to (99.8, 153.5)
- moved TP4 111.9 mm to (88.9, 153.5)
- moved SW4 55.0 mm to (198.8, 125.7)
- moved D5 37.7 mm to (118.9, 150.7), turned to 0 degrees
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- renumbered TP55 to CLK, TP54 to DATA
Connections:
- SW3 pad 1: Net-(J5-Pad1) -> /PSU/PMOSReversePolarityProtection/VIN
- SW3 pad 2: /PSU/PMOSReversePolarityProtection/VIN -> Net-(J5-Pad1)
Routing:
- net +5V: track 292.8 -> 188.4 mm
- net /PSU/TPS563200_BUCK_MISC/BUCK_VIN: track 165.7 -> 79.6 mm
- net +3V3: track 335.4 -> 380.3 mm, vias 9 -> 12
- net /CrossPoint Output Switching/X7: track 22.5 -> 67.0 mm
- net /Input Keyscan and RGB LED Driver/KEY_C0: track 261.8 -> 301.7 mm
- net /Input Keyscan and RGB LED Driver/KEY_C2: track 265.8 -> 305.5 mm
- net /Input Keyscan and RGB LED Driver/ADP5587_WRITE: track 93.0 -> 55.4 mm, vias 1 -> 2
- net Net-(R21-Pad2): track 240.0 -> 273.6 mm, vias 4 -> 2
- net /MCU/SPI2_MOSI: track 222.5 -> 252.5 mm
- net /OLED_Display/RESET: track 107.3 -> 77.5 mm, vias 1 -> 0
- net /OLED_Display/CLK: track 107.2 -> 78.5 mm, vias 1 -> 0
- net /OLED_Display/DATA: track 106.5 -> 77.8 mm, vias 1 -> 0
- net /MCU/SPI2_GSCLK: track 113.7 -> 86.7 mm, vias 3 -> 2
- net /MCU/SPI2_LAT: track 121.0 -> 96.1 mm, vias 1 -> 3
- net /CrossPoint Output Switching/ADG2188_SDA: track 24.8 -> 48.6 mm, vias 1 -> 3
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Other:
- board size 250.2 x 99.1 mm -> 249.6 x 122.6 mm
- board text added: "0000: 0 0001: 1 0010: 2 0011: 3 0100: 4 0101: 5 0110: 6 0111: 7"
- board text added: "1000: 8 1001: 9 1010: 10 1011: 11 1100: 12 1101: 13 1110: 14 1111: 15"
- board text added: "3.3V"
- board text added: "3.3V OLED"
- board text added: "5V"
- board text added: "5V OLED"
- board text added: "5V RGB"
- board text added: "ADJUST"
- board text added: "CLEAR"
- board text added: "CLK"
- board text added: "CS"
- board text added: "D/C"
- board text added: "GSCLK"
- board text added: "INT"
- board text added: "KEY C0"
- board text added: "KEY C1"
- board text added: "KEY C2"
- board text added: "KEY C3"
- board text added: "KEY R0"
- board text added: "KEY R1"
- board text added: "KEY R2"
- board text added: "KEY R3"
- board text added: "KEY R4"
- board text added: "KEY R5"
- board text added: "KEY R6"
- board text added: "KEY R7"
- board text added: "LAT"
- board text added: "MIDI CHANNEL"
- board text added: "MIDI RX"
- board text added: "MIDI TX"
- board text added: "OFF"
- board text added: "ON"
- board text added: "PRESET WRITE"
- board text added: "RST"
- board text added: "SCL"
- board text added: "SDA"
- board text added: "SIN"
- board text added: "SOUT"
- board text added: "WRITE PROTECT"
- board text added: "X0"
- board text added: "X1"
- board text added: "X2"
- board text added: "X3"
- board text added: "X4"
- board text added: "X5"
- board text added: "X6"
- board text added: "X7"
- board text added: "Y1"
- board text added: "Y2"
- board text added: "Y3"
- board text added: "Y4"
- board text added: "Y5"
- board text added: "Y6"
- board text added: "Y7"

Commit message: updated
Parts:
- removed TP1, TP51: TestPoint, TestPoint:TestPoint_Pad_D1.0mm
- added D7: RED, LED_SMD:LED_0805_2012Metric_Pad1.15x1.40mm_HandSolder, F.Cu at (98.6, 128.0)
- added R13: 2K2, Resistor_SMD:R_0805_2012Metric_Pad1.20x1.40mm_HandSolder, F.Cu at (102.6, 128.0)
- added REF**: MountingHole_3.2mm_M3_Pad_Via, MountingHole:MountingHole_3.2mm_M3_Pad_Via, F.Cu at (325.8, 161.3)
- added REF**: MountingHole_3.2mm_M3_Pad_Via, MountingHole:MountingHole_3.2mm_M3_Pad_Via, F.Cu at (86.4, 161.3)
- R5: footprint Resistor_SMD:R_0805_2012Metric_Pad1.20x1.40mm_HandSolder -> Resistor_SMD:R_1206_3216Metric_Pad1.30x1.75mm_HandSolder
- U35: footprint Package_CSP:LFCSP-24-1EP_4x4mm_P0.5mm_EP2.3x2.3mm -> Package_CSP:LFCSP-24-1EP_4x4mm_P0.5mm_EP2.3x2.3mm_ThermalVias
- moved TP3 18.0 mm to (88.1, 117.1)
- moved SW4 5.84 mm to (198.6, 119.9)
- moved TP28 5.09 mm to (257.6, 159.8)
- moved TP27 4.57 mm to (246.4, 160.0)
- moved R5 4.44 mm to (88.6, 121.4), turned to 180 degrees
- moved D1 3.54 mm to (87.1, 127.8)
- moved TP25 3.30 mm to (217.8, 160.0)
- moved Q1 3.07 mm to (91.7, 127.8)
- moved SW3 2.54 mm to (98.6, 119.4)
- moved TP18 2.03 mm to (315.6, 159.9)
- moved TP4 1.91 mm to (87.0, 153.5)
- moved U17 0.05 mm to (93.4, 176.1)
- renumbered Y0 to TP49, DATA to TP54, CLK to TP55
Routing:
- net /MCU/SPI2_MOSI: track 252.5 -> 102.4 mm
- net Net-(R21-Pad2): track 273.6 -> 242.6 mm, vias 2 -> 5
- net /CrossPoint Output Switching/X7: track 67.0 -> 44.3 mm
- net /PSU/+5V_RGB: track 119.7 -> 133.3 mm
- net /CrossPoint Output Switching/X3: track 39.0 -> 26.3 mm, vias 1 -> 2
- net /MCU/TIM1_CH2: track 196.1 -> 187.3 mm
- net /PSU/TPS563200_BUCK_MISC/BUCK_VIN: track 79.6 -> 88.4 mm
- net /Input Keyscan and RGB LED Driver/KEY_C3: track 330.9 -> 336.8 mm
- net /Input Keyscan and RGB LED Driver/DIPSW2: track 25.1 -> 30.9 mm
- net /Input Keyscan and RGB LED Driver/DIPSW4: track 29.5 -> 35.3 mm
- net /Input Keyscan and RGB LED Driver/DIPSW3: track 27.3 -> 33.1 mm
- net /Input Keyscan and RGB LED Driver/DIPSW1: track 22.5 -> 28.3 mm
- net GND: track 47.0 -> 42.1 mm, vias 75 -> 265
- net /Input Keyscan and RGB LED Driver/KEY_C0: track 301.7 -> 305.8 mm
- net Net-(D7-Pad1): track 0.00 -> 4.07 mm
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- added copper zone on F.Cu, net /PSU/TPS563200_BUCK_MISC/BUCK_VIN
- added copper zone on B.Cu, net Net-(SW3-Pad3)
- added copper zone on F.Cu, net Net-(SW3-Pad3)
Other:
- board text added: "9-15V 4A"
- board text added: "BassStation Sequencer RevA"
- board text added: "WRITE PRESET"
- board text removed: "PRESET WRITE"
