File: SequencerMidiController/MIDI.sch (KiCad schematic (older format))
At the start: 13 parts, among them J1 MIDI IN, J2 MIDI OUT, U42 74LVC1G34, U43 6N135S

Commit message: Completed RevA layout
Other:
- moved on the sheet: J2, R2, R3, TP50, TP51, U42
Changed lines of the file:
@@
 L MidiDin5:DIN-5 J2
 U 1 1 60BA1755
-P 7025 3900
-F 0 "J2" V 6979 3670 50  0000 R CNN
-F 1 "MIDI OUT" V 7070 3670 50  0000 R CNN
-F 2 "RS_5P180_DIN5_SOCKET_WSHIELD:RS_5P180_DIN5_SOCKET_WSHIELD" H 7025 3900 50  0001 C CNN
-F 3 "~" H 7025 3900 50  0001 C CNN
-F 4 "~" H 7025 3900 50  0001 C CNN "LcscNo"
-F 5 "~" H 7025 3900 50  0001 C CNN "Type"
-	1    7025 3900
+P 7150 4725
+F 0 "J2" V 7104 4495 50  0000 R CNN
+F 1 "MIDI OUT" V 7195 4495 50  0000 R CNN
+F 2 "RS_5P180_DIN5_SOCKET_WSHIELD:RS_5P180_DIN5_SOCKET_WSHIELD" H 7150 4725 50  0001 C CNN
+F 3 "~" H 7150 4725 50  0001 C CNN
+F 4 "~" H 7150 4725 50  0001 C CNN "LcscNo"
+F 5 "~" H 7150 4725 50  0001 C CNN "Type"
+	1    7150 4725
 	0    -1   1    0
 $EndComp
-NoConn ~ 6725 3900
-NoConn ~ 7125 3600
-NoConn ~ 7125 4200
+NoConn ~ 6850 4725
+NoConn ~ 7250 4425
+NoConn ~ 7250 5025
 $Comp
 L Device:R R3
 U 1 1 60BA2841
-P 6925 3325
-F 0 "R3" H 6855 3279 50  0000 R CNN
-F 1 "220R" H 6855 3370 50  0000 R CNN
-F 2 "Resistor_SMD:R_0805_2012Metric_Pad1.20x1.40mm_HandSolder" V 6855 3325 50  0001 C CNN
-F 3 "~" H 6925 3325 50  0001 C CNN
-F 4 "~" H 6925 3325 50  0001 C CNN "LcscNo"
-F 5 "~" H 6925 3325 50  0001 C CNN "Type"
-	1    6925 3325
+P 7050 4150
+F 0 "R3" H 6980 4104 50  0000 R CNN
+F 1 "220R" H 6980 4195 50  0000 R CNN
+F 2 "Resistor_SMD:R_0805_2012Metric_Pad1.20x1.40mm_HandSolder" V 6980 4150 50  0001 C CNN
+F 3 "~" H 7050 4150 50  0001 C CNN
+F 4 "~" H 7050 4150 50  0001 C CNN "LcscNo"
+F 5 "~" H 7050 4150 50  0001 C CNN "Type"
+	1    7050 4150
 	1    0    0    1
 $EndComp
 Wire Wire Line
-	6925 3475 6925 3600
+	7050 4300 7050 4425
 $Comp
 L Device:R R2
 U 1 1 60BAC1D0
-P 5775 4375
-F 0 "R2" V 5568 4375 50  0000 C CNN
-F 1 "220R" V 5659 4375 50  0000 C CNN
-F 2 "Resistor_SMD:R_0805_2012Metric_Pad1.20x1.40mm_HandSolder" V 5705 4375 50  0001 C CNN
-F 3 "~" H 5775 4375 50  0001 C CNN
-F 4 "~" H 5775 4375 50  0001 C CNN "LcscNo"
-F 5 "~" H 5775 4375 50  0001 C CNN "Type"
-	1    5775 4375
+P 5900 5200
+F 0 "R2" V 5693 5200 50  0000 C CNN
+F 1 "220R" V 5784 5200 50  0000 C CNN
+F 2 "Resistor_SMD:R_0805_2012Metric_Pad1.20x1.40mm_HandSolder" V 5830 5200 50  0001 C CNN
+F 3 "~" H 5900 5200 50  0001 C CNN
+F 4 "~" H 5900 5200 50  0001 C CNN "LcscNo"
+F 5 "~" H 5900 5200 50  0001 C CNN "Type"
+	1    5900 5200
 	0    -1   1    0
 $EndComp
 Wire Wire Line
-	5925 4375 6325 4375
+	6050 5200 6450 5200
 Wire Wire Line
 	7200 1950 7700 1950
 Wire Wire Line
-	6925 4200 6925 4375
+	7050 5025 7050 5200
 $Comp
 L 74xGxx:74LVC1G34 U42
 U 1 1 60BC14F0
-P 4925 4375
-F 0 "U42" H 4425 4650 50  0000 C CNN
-F 1 "74LVC1G34" H 4575 4550 50  0000 C CNN
-F 2 "Package_TO_SOT_SMD:SOT-23-5_HandSoldering" H 4925 4375 50  0001 C CNN
-F 3 "http://www.ti.com/lit/sg/scyt129e/scyt129e.pdf" H 4925 4375 50  0001 C CNN
-F 4 "~" H 4925 4375 50  0001 C CNN "LcscNo"
-F 5 "~" H 4925 4375 50  0001 C CNN "Type"
-	1    4925 4375
+P 5050 5200
+F 0 "U42" H 4550 5475 50  0000 C CNN
+F 1 "74LVC1G34" H 4700 5375 50  0000 C CNN
+F 2 "Package_TO_SOT_SMD:SOT-23-5_HandSoldering" H 5050 5200 50  0001 C CNN
+F 3 "http://www.ti.com/lit/sg/scyt129e/scyt129e.pdf" H 5050 5200 50  0001 C CNN
+F 4 "~" H 5050 5200 50  0001 C CNN "LcscNo"
+F 5 "~" H 5050 5200 50  0001 C CNN "Type"
+	1    5050 5200
 	1    0    0    -1
 $EndComp
 Wire Wire Line
-	4625 4375 3950 4375
-Text HLabel 3750 4375 0    50   Input ~ 0
+	4750 5200 4075 5200
+Text HLabel 3875 5200 0    50   Input ~ 0
 MIDI_TX
 Wire Wire Line
-	5175 4375 5625 4375
+	5300 5200 5750 5200
 Text HLabel 6375 1125 0    50   Input ~ 0
 MIDI_VIN
 Wire Wire Line
 	6375 1125 6525 1125
-Text HLabel 6825 2925 0    50   Input ~ 0
+Text HLabel 6950 3750 0    50   Input ~ 0
 MIDI_VIN
 Wire Wire Line
-	6825 2925 6925 2925
+	6950 3750 7050 3750
 Wire Wire Line
-	6925 2925 6925 3175
+	7050 3750 7050 4000
 Wire Wire Line
-	4925 4275 4925 4075
+	5050 5100 5050 4900
 $Comp
 L power:+3.3V #PWR0101
 U 1 1 68A59BBA
-P 4925 4075
-F 0 "#PWR0101" H 4925 3925 50  0001 C CNN
-F 1 "+3.3V" H 4940 4248 50  0000 C CNN
-F 2 "" H 4925 4075 50  0001 C CNN
-F 3 "" H 4925 4075 50  0001 C CNN
-	1    4925 4075
+P 5050 4900
+F 0 "#PWR0101" H 5050 4750 50  0001 C CNN
+F 1 "+3.3V" H 5065 5073 50  0000 C CNN
+F 2 "" H 5050 4900 50  0001 C CNN
+F 3 "" H 5050 4900 50  0001 C CNN
+	1    5050 4900
 	1    0    0    -1
 $EndComp
@@
 L power:GNDS #PWR0103
 U 1 1 68A5A228
-P 4925 4625
-F 0 "#PWR0103" H 4925 4375 50  0001 C CNN
-F 1 "GNDS" H 4930 4452 50  0000 C CNN
-F 2 "" H 4925 4625 50  0001 C CNN
-F 3 "" H 4925 4625 50  0001 C CNN
-	1    4925 4625
+P 5050 5450
+F 0 "#PWR0103" H 5050 5200 50  0001 C CNN
+F 1 "GNDS" H 5055 5277 50  0000 C CNN
+F 2 "" H 5050 5450 50  0001 C CNN
+F 3 "" H 5050 5450 50  0001 C CNN
+	1    5050 5450
 	1    0    0    -1
 $EndComp
 Wire Wire Line
-	4925 4625 4925 4475
+	5050 5450 5050 5300
 $Comp
 L Connector:TestPoint TP50
 U 1 1 63B85270
-P 3950 4250
-F 0 "TP50" H 4008 4322 50  0000 L CNN
-F 1 "TestPoint" H 4008 4277 50  0001 L CNN
-F 2 "TestPoint:TestPoint_Pad_D1.0mm" H 4150 4250 50  0001 C CNN
-F 3 "~" H 4150 4250 50  0001 C CNN
-F 4 "~" H 3950 4250 50  0001 C CNN "LcscNo"
-F 5 "~" H 3950 4250 50  0001 C CNN "Type"
-	1    3950 4250
+P 4075 5075
+F 0 "TP50" H 4133 5147 50  0000 L CNN
+F 1 "TestPoint" H 4133 5102 50  0001 L CNN
+F 2 "TestPoint:TestPoint_Pad_D1.0mm" H 4275 5075 50  0001 C CNN
+F 3 "~" H 4275 5075 50  0001 C CNN
+F 4 "~" H 4075 5075 50  0001 C CNN "LcscNo"
+F 5 "~" H 4075 5075 50  0001 C CNN "Type"
+	1    4075 5075
 	1    0    0    -1
 $EndComp
 Wire Wire Line
-	3950 4250 3950 4375
-Connection ~ 3950 4375
+	4075 5075 4075 5200
+Connection ~ 4075 5200
 Wire Wire Line
-	3950 4375 3750 4375
+	4075 5200 3875 5200
 $Comp
 L Connector:TestPoint TP51
 U 1 1 63B85A0C
-P 6325 4250
-F 0 "TP51" H 6383 4322 50  0000 L CNN
-F 1 "TestPoint" H 6383 4277 50  0001 L CNN
-F 2 "TestPoint:TestPoint_Pad_D1.0mm" H 6525 4250 50  0001 C CNN
-F 3 "~" H 6525 4250 50  0001 C CNN
-F 4 "~" H 6325 4250 50  0001 C CNN "LcscNo"
-F 5 "~" H 6325 4250 50  0001 C CNN "Type"
-	1    6325 4250
+P 6450 5075
+F 0 "TP51" H 6508 5147 50  0000 L CNN
+F 1 "TestPoint" H 6508 5102 50  0001 L CNN
+F 2 "TestPoint:TestPoint_Pad_D1.0mm" H 6650 5075 50  0001 C CNN
+F 3 "~" H 6650 5075 50  0001 C CNN
+F 4 "~" H 6450 5075 50  0001 C CNN "LcscNo"
+F 5 "~" H 6450 5075 50  0001 C CNN "Type"
+	1    6450 5075
 	1    0    0    -1
 $EndComp
 Wire Wire Line
-	6325 4250 6325 4375
-Connection ~ 6325 4375
+	6450 5075 6450 5200
+Connection ~ 6450 5200
 Wire Wire Line
-	6325 4375 6925 4375
+	6450 5200 7050 5200
 $EndSCHEMATC

Commit message: updated
Parts:
- removed TP1, TP51: TestPoint, TestPoint:TestPoint_Pad_D1.0mm, symbol Connector:TestPoint
Changed lines of the file:
@@
 	3400 1575 3400 1500
-Wire Wire Line
-	3400 1500 3675 1500
 Wire Wire Line
 	4600 1725 4600 1500
@@
 Connection ~ 7200 1950
 $Comp
-L Connector:TestPoint TP1
-U 1 1 60BA126E
-P 3675 1375
-F 0 "TP1" H 3733 1447 50  0000 L CNN
-F 1 "TestPoint" H 3733 1402 50  0001 L CNN
-F 2 "TestPoint:TestPoint_Pad_D1.0mm" H 3875 1375 50  0001 C CNN
-F 3 "~" H 3875 1375 50  0001 C CNN
-F 4 "~" H 3675 1375 50  0001 C CNN "LcscNo"
-F 5 "~" H 3675 1375 50  0001 C CNN "Type"
-	1    3675 1375
-	1    0    0    -1
-$EndComp
-Wire Wire Line
-	3675 1375 3675 1500
-Connection ~ 3675 1500
-Wire Wire Line
-	3675 1500 3975 1500
-$Comp
 L MidiDin5:DIN-5 J2
 U 1 1 60BA1755
@@
 $EndComp
 Wire Wire Line
-	6050 5200 6450 5200
-Wire Wire Line
 	7200 1950 7700 1950
 Wire Wire Line
@@
 Wire Wire Line
 	4075 5200 3875 5200
-$Comp
-L Connector:TestPoint TP51
-U 1 1 63B85A0C
-P 6450 5075
-F 0 "TP51" H 6508 5147 50  0000 L CNN
-F 1 "TestPoint" H 6508 5102 50  0001 L CNN
-F 2 "TestPoint:TestPoint_Pad_D1.0mm" H 6650 5075 50  0001 C CNN
-F 3 "~" H 6650 5075 50  0001 C CNN
-F 4 "~" H 6450 5075 50  0001 C CNN "LcscNo"
-F 5 "~" H 6450 5075 50  0001 C CNN "Type"
-	1    6450 5075
-	1    0    0    -1
-$EndComp
-Wire Wire Line
-	6450 5075 6450 5200
-Connection ~ 6450 5200
-Wire Wire Line
-	6450 5200 7050 5200
+Wire Wire Line
+	3400 1500 3975 1500
+Wire Wire Line
+	6050 5200 7050 5200
 $EndSCHEMATC
