File: SequencerMidiController/PSU.sch (KiCad schematic (older format))
At the start: 2 parts, among them J5 Barrel_Jack_Switch, SW3 SW_SPST

Commit message: Completed RevA layout
Parts:
- SW3: footprint Connector_Molex:Molex_KK-254_AE-6410-02A_1x02_P2.54mm_Vertical -> DailywellSwitches:Dailywell_SPDT; symbol Switch:SW_SPST -> Switch:SW_SPDT
Connections:
- net PMOSReversePolarityProtection/VIN: now also SW3.1 (A); no longer SW3.2 (B)
- net at J5.1: now also SW3.2 (B); no longer SW3.1 (A)
- no-connect marks 0 -> 1
Other:
- moved on the sheet: J5
Changed lines of the file:
@@
 L Connector:Barrel_Jack_Switch J5
 U 1 1 60BD4034
-P 1475 1875
-F 0 "J5" H 1532 2192 50  0000 C CNN
-F 1 "Barrel_Jack_Switch" H 1532 2101 50  0000 C CNN
-F 2 "Connector_BarrelJack:BarrelJack_Horizontal" H 1525 1835 50  0001 C CNN
-F 3 "~" H 1525 1835 50  0001 C CNN
-F 4 "~" H 1475 1875 50  0001 C CNN "LcscNo"
-F 5 "~" H 1475 1875 50  0001 C CNN "Type"
-	1    1475 1875
+P 1475 1975
+F 0 "J5" H 1532 2292 50  0000 C CNN
+F 1 "Barrel_Jack_Switch" H 1532 2201 50  0000 C CNN
+F 2 "Connector_BarrelJack:BarrelJack_Horizontal" H 1525 1935 50  0001 C CNN
+F 3 "~" H 1525 1935 50  0001 C CNN
+F 4 "~" H 1475 1975 50  0001 C CNN "LcscNo"
+F 5 "~" H 1475 1975 50  0001 C CNN "Type"
+	1    1475 1975
 	1    0    0    -1
 $EndComp
 Wire Wire Line
-	1775 1775 2800 1775
+	1775 1875 2800 1875
 Wire Wire Line
-	1775 1875 2300 1875
+	1775 1975 2300 1975
 Wire Wire Line
-	2300 1875 2300 1975
+	2300 1975 2300 2075
 $Comp
 L power:GNDS #PWR0104
 U 1 1 60BD50AE
-P 2300 2375
-F 0 "#PWR0104" H 2300 2125 50  0001 C CNN
-F 1 "GNDS" H 2305 2202 50  0000 C CNN
-F 2 "" H 2300 2375 50  0001 C CNN
-F 3 "" H 2300 2375 50  0001 C CNN
-	1    2300 2375
+P 2300 2475
+F 0 "#PWR0104" H 2300 2225 50  0001 C CNN
+F 1 "GNDS" H 2305 2302 50  0000 C CNN
+F 2 "" H 2300 2475 50  0001 C CNN
+F 3 "" H 2300 2475 50  0001 C CNN
+	1    2300 2475
 	1    0    0    -1
 $EndComp
 Wire Wire Line
-	1775 1975 2300 1975
-Connection ~ 2300 1975
+	1775 2075 2300 2075
+Connection ~ 2300 2075
 Wire Wire Line
-	2300 1975 2300 2375
+	2300 2075 2300 2475
 $Sheet
 S 5725 1450 1275 700
@@
 	7875 3075 9925 3075
 $Comp
-L Switch:SW_SPST SW3
+L Switch:SW_SPDT SW3
 U 1 1 63B8B2DD
-P 3000 1775
-F 0 "SW3" H 3000 2010 50  0000 C CNN
-F 1 "SW_SPST" H 3000 1919 50  0000 C CNN
-F 2 "Connector_Molex:Molex_KK-254_AE-6410-02A_1x02_P2.54mm_Vertical" H 3000 1775 50  0001 C CNN
-F 3 "~" H 3000 1775 50  0001 C CNN
-F 4 "~" H 3000 1775 50  0001 C CNN "LcscNo"
-F 5 "~" H 3000 1775 50  0001 C CNN "Type"
-	1    3000 1775
+P 3000 1875
+F 0 "SW3" H 3000 2110 50  0000 C CNN
+F 1 "SW_SPST" H 3000 2019 50  0000 C CNN
+F 2 "DailywellSwitches:Dailywell_SPDT" H 3000 1875 50  0001 C CNN
+F 3 "~" H 3000 1875 50  0001 C CNN
+F 4 "~" H 3000 1875 50  0001 C CNN "LcscNo"
+F 5 "~" H 3000 1875 50  0001 C CNN "Type"
+	1    3000 1875
 	1    0    0    -1
 $EndComp
@@
 L power:PWR_FLAG #FLG0105
 U 1 1 68A724DD
-P 2300 1975
-F 0 "#FLG0105" H 2300 2050 50  0001 C CNN
-F 1 "PWR_FLAG" V 2300 2325 50  0000 C CNN
-F 2 "" H 2300 1975 50  0001 C CNN
-F 3 "~" H 2300 1975 50  0001 C CNN
-	1    2300 1975
+P 2300 2075
+F 0 "#FLG0105" H 2300 2150 50  0001 C CNN
+F 1 "PWR_FLAG" V 2300 2425 50  0000 C CNN
+F 2 "" H 2300 2075 50  0001 C CNN
+F 3 "~" H 2300 2075 50  0001 C CNN
+	1    2300 2075
 	0    1    1    0
 $EndComp
+NoConn ~ 3200 1975
 $EndSCHEMATC

Commit message: updated
Other:
- note added: "9-15V\n"
Changed lines of the file:
@@
 $EndComp
 NoConn ~ 3200 1975
+Text Notes 1400 1475 0    50   ~ 0
+9-15V\n
 $EndSCHEMATC
