File: SequencerMidiController/SequencerInputs.sch (KiCad schematic (older format))
At the start: 42 parts, among them SW4 SW_SPDT-2MS1T1B1M2QES, SW5 SW_SPST, SW6 SW_DIP_x04, U35 ADP5587-ACPZ_LFCSP24, U36 TLC5955DCA_HTSSOP56, U37 TLC5955DCA_HTSSOP56

Commit message: RevA Layout draft completed
- Needs tidy up
- Add test points
Parts:
- removed R13, R15, R16, R17, R31: 220R, Resistor_SMD:R_0805_2012Metric_Pad1.20x1.40mm_HandSolder, symbol Device:R
- removed SW4: SW_SPDT-2MS1T1B1M2QES, DailywellSwitches:Dailywell_SPDT, symbol Switch:SW_SPDT
- removed SW6: SW_DIP_x04, Button_Switch_THT:SW_DIP_SPSTx04_Slide_9.78x12.34mm_W7.62mm_P2.54mm, symbol Switch:SW_DIP_x04
- added SW2: SW_SPDT-2MS1T1B1M2QES, DailywellSwitches:Dailywell_SPDT, symbol Switch:SW_SPDT
- added SW4: SW_DIP_x04, Button_Switch_THT:SW_DIP_SPSTx04_Slide_9.78x12.34mm_W7.62mm_P2.54mm, symbol Switch:SW_DIP_x04
- R20: value 100R -> 220R
- SW5: footprint Button_Switch_THT:SW_TH_Tactile_Omron_B3F-10xx -> Button_Switch_THT:SW_PUSH-12mm
Connections:
- net +3V3 is gone; now on net ADP5587_VIN: C8.1, R10.2, R14.1, R18.2, R19.1, R30.2, U35.21 (VCC)
- net ADP5587_VIN: now also R20.2
- net ADP5587_WRITE: now also R20.1; no longer R30.1
- net ADP5587_WRITEPROTECT: now also SW2.2 (B)
- net DIPSW1: now also SW4.1
- net DIPSW2: now also SW4.2
- net DIPSW3: now also SW4.3
- net DIPSW4: now also SW4.4
- net GNDS: now also SW2.1 (A), SW4.5, SW4.6, SW4.7, SW4.8; no longer R20.1
- net OUTB1 renamed LEDBK10
- net OUTB10 renamed LEDBK6
- net OUTB11 renamed LEDBK3
- net OUTB12 renamed LEDBK1
- net OUTB13 renamed LEDBK7
- net OUTB14 renamed LEDBK5
- net OUTB15 renamed LEDBK4
- net OUTB16 renamed LEDBK2
- net OUTB17 renamed LEDBK31
- net OUTB18 renamed LEDBK29
- net OUTB19 renamed LEDBK28
- net OUTB2 renamed LEDBK12
- net OUTB20 renamed LEDBK26
- net OUTB21 renamed LEDBK32
- net OUTB22 renamed LEDBK30
- net OUTB23 renamed LEDBK27
- net OUTB24 renamed LEDBK25
- net OUTB25 renamed LEDBK17
- net OUTB26 renamed LEDBK19
- net OUTB27 renamed LEDBK22
- net OUTB28 renamed LEDBK24
- net OUTB29 renamed LEDBK18
- net OUTB3 renamed LEDBK13
- net OUTB30 renamed LEDBK20
- net OUTB31 renamed LEDBK21
- net OUTB32 renamed LEDBK23
- net OUTB4 renamed LEDBK15
- net OUTB5 renamed LEDBK9
- net OUTB6 renamed LEDBK11
- net OUTB7 renamed LEDBK14
- net OUTB8 renamed LEDBK16
- net OUTB9 renamed LEDBK8
- net OUTG1 renamed LEDGK10
- net OUTG10 renamed LEDGK6
- net OUTG11 renamed LEDGK3
- net OUTG12 renamed LEDGK1
- net OUTG13 renamed LEDGK7
- net OUTG14 renamed LEDGK5
- net OUTG15 renamed LEDGK4
- net OUTG16 renamed LEDGK2
- net OUTG17 renamed LEDGK31
- net OUTG18 renamed LEDGK29
- net OUTG19 renamed LEDGK28
- net OUTG2 renamed LEDGK12
- net OUTG20 renamed LEDGK26
- net OUTG21 renamed LEDGK32
- net OUTG22 renamed LEDGK30
- net OUTG23 renamed LEDGK27
- net OUTG24 renamed LEDGK25
- net OUTG25 renamed LEDGK17
- net OUTG26 renamed LEDGK19
- net OUTG27 renamed LEDGK22
- net OUTG28 renamed LEDGK24
- net OUTG29 renamed LEDGK18
- net OUTG3 renamed LEDGK13
- net OUTG30 renamed LEDGK20
- net OUTG31 renamed LEDGK21
- net OUTG32 renamed LEDGK23
- net OUTG4 renamed LEDGK15
- net OUTG5 renamed LEDGK9
- net OUTG6 renamed LEDGK11
- net OUTG7 renamed LEDGK14
- net OUTG8 renamed LEDGK16
- net OUTG9 renamed LEDGK8
- net OUTR1 renamed LEDRK10
- net OUTR10 renamed LEDRK6
- net OUTR11 renamed LEDRK3
- net OUTR12 renamed LEDRK1
- net OUTR13 renamed LEDRK7
- net OUTR14 renamed LEDRK5
- net OUTR15 renamed LEDRK4
- net OUTR16 renamed LEDRK2
- net OUTR17 renamed LEDRK31
- net OUTR18 renamed LEDRK29
- net OUTR19 renamed LEDRK28
- net OUTR2 renamed LEDRK12
- net OUTR20 renamed LEDRK26
- net OUTR21 renamed LEDRK32
- net OUTR22 renamed LEDRK30
- net OUTR23 renamed LEDRK27
- net OUTR24 renamed LEDRK25
- net OUTR25 renamed LEDRK17
- net OUTR26 renamed LEDRK19
- net OUTR27 renamed LEDRK22
- net OUTR28 renamed LEDRK24
- net OUTR29 renamed LEDRK18
- net OUTR3 renamed LEDRK13
- net OUTR30 renamed LEDRK20
- net OUTR31 renamed LEDRK21
- net OUTR32 renamed LEDRK23
- net OUTR4 renamed LEDRK15
- net OUTR5 renamed LEDRK9
- net OUTR6 renamed LEDRK11
- net OUTR7 renamed LEDRK14
- net OUTR8 renamed LEDRK16
- net OUTR9 renamed LEDRK8
- new net: R30.1, SW2.3 (C)
Other:
- note removed: "Use if sw_dip sinks\nexcessive current"
- moved on the sheet: TP22, TP23

Commit message: Completed RevA layout
Parts:
- removed TP12, TP14: TestPoint, TestPoint:TestPoint_Pad_D1.0mm, symbol Connector:TestPoint
Connections:
- net TLC5955_LAT: no longer TP16.1
- net at U36.28 (SOUT), U37.1 (SIN): now also TP16.1
Other:
- moved on the sheet: TP16
Changed lines of the file:
@@
 	1    0    0    -1
 $EndComp
-Wire Wire Line
-	3775 20300 2450 20300
 NoConn ~ 5425 20300
 Wire Wire Line
@@
 	4100 15925 3825 15925
 Wire Wire Line
-	1450 20500 3775 20500
+	1450 20500 2700 20500
 Wire Wire Line
 	1450 20500 1450 15300
@@
 	1    0    0    -1
 $EndComp
-Wire Wire Line
-	2450 20300 2450 19900
-$Comp
-L Connector:TestPoint TP?
-U 1 1 61819693
-P 2450 19900
-AR Path="/60BD3123/60BD5AA5/61819693" Ref="TP?"  Part="1"
-AR Path="/60BD3123/63615DFB/61819693" Ref="TP?"  Part="1"
-AR Path="/60BCDD64/61819693" Ref="TP12"  Part="1"
-F 0 "TP12" H 2375 20150 50  0000 L CNN
-F 1 "TestPoint" H 2508 19927 50  0001 L CNN
-F 2 "TestPoint:TestPoint_Pad_D1.0mm" H 2650 19900 50  0001 C CNN
-F 3 "~" H 2650 19900 50  0001 C CNN
-F 4 "~" H 2450 19900 50  0001 C CNN "LcscNo"
-F 5 "~" H 2450 19900 50  0001 C CNN "Type"
-	1    2450 19900
-	1    0    0    -1
-$EndComp
-Wire Wire Line
-	2575 20400 2575 20025
-$Comp
-L Connector:TestPoint TP?
-U 1 1 61895ED5
-P 2575 20025
-AR Path="/60BD3123/60BD5AA5/61895ED5" Ref="TP?"  Part="1"
-AR Path="/60BD3123/63615DFB/61895ED5" Ref="TP?"  Part="1"
-AR Path="/60BCDD64/61895ED5" Ref="TP14"  Part="1"
-F 0 "TP14" H 2500 20275 50  0000 L CNN
-F 1 "TestPoint" H 2633 20052 50  0001 L CNN
-F 2 "TestPoint:TestPoint_Pad_D1.0mm" H 2775 20025 50  0001 C CNN
-F 3 "~" H 2775 20025 50  0001 C CNN
-F 4 "~" H 2575 20025 50  0001 C CNN "LcscNo"
-F 5 "~" H 2575 20025 50  0001 C CNN "Type"
-	1    2575 20025
-	1    0    0    -1
-$EndComp
 $Comp
 L Connector:TestPoint TP?
 U 1 1 61A0DA66
-P 2700 19900
+P 2700 19800
 AR Path="/60BD3123/60BD5AA5/61A0DA66" Ref="TP?"  Part="1"
 AR Path="/60BD3123/63615DFB/61A0DA66" Ref="TP?"  Part="1"
 AR Path="/60BCDD64/61A0DA66" Ref="TP16"  Part="1"
-F 0 "TP16" H 2625 20150 50  0000 L CNN
-F 1 "TestPoint" H 2758 19927 50  0001 L CNN
-F 2 "TestPoint:TestPoint_Pad_D1.0mm" H 2900 19900 50  0001 C CNN
-F 3 "~" H 2900 19900 50  0001 C CNN
-F 4 "~" H 2700 19900 50  0001 C CNN "LcscNo"
-F 5 "~" H 2700 19900 50  0001 C CNN "Type"
-	1    2700 19900
-	1    0    0    -1
-$EndComp
-Wire Wire Line
-	2700 19900 2700 20600
+F 0 "TP16" H 2625 20050 50  0000 L CNN
+F 1 "TestPoint" H 2758 19827 50  0001 L CNN
+F 2 "TestPoint:TestPoint_Pad_D1.0mm" H 2900 19800 50  0001 C CNN
+F 3 "~" H 2900 19800 50  0001 C CNN
+F 4 "~" H 2700 19800 50  0001 C CNN "LcscNo"
+F 5 "~" H 2700 19800 50  0001 C CNN "Type"
+	1    2700 19800
+	1    0    0    -1
+$EndComp
+Wire Wire Line
+	2700 19800 2700 20500
 Wire Wire Line
 	4650 3125 4650 2975
@@
 Wire Wire Line
 	2000 14275 2675 14275
-Connection ~ 2450 20300
-Connection ~ 2575 20400
-Wire Wire Line
-	2575 20400 3775 20400
-Connection ~ 2700 20600
-Wire Wire Line
-	2700 20600 3775 20600
-Wire Wire Line
-	2250 20400 2575 20400
-Wire Wire Line
-	2250 20600 2700 20600
-Wire Wire Line
-	2250 20300 2450 20300
 Text Label 6175 20000 2    50   ~ 0
 LEDBK23
@@
 	-1   0    0    -1
 $EndComp
+Wire Wire Line
+	2250 20300 3775 20300
+Wire Wire Line
+	2250 20400 3775 20400
+Connection ~ 2700 20500
+Wire Wire Line
+	2700 20500 3775 20500
+Wire Wire Line
+	2250 20600 3775 20600
 $EndSCHEMATC

Commit message: updated
Parts:
- U35: footprint Package_CSP:LFCSP-24-1EP_4x4mm_P0.5mm_EP2.3x2.3mm -> Package_CSP:LFCSP-24-1EP_4x4mm_P0.5mm_EP2.3x2.3mm_ThermalVias
Changed lines of the file:
@@
 F 0 "U35" H 6475 4850 50  0000 C CNN
 F 1 "ADP5587-ACPZ_LFCSP24" H 5500 2725 50  0000 C CNN
-F 2 "Package_CSP:LFCSP-24-1EP_4x4mm_P0.5mm_EP2.3x2.3mm" H 6675 4375 50  0001 C CNN
+F 2 "Package_CSP:LFCSP-24-1EP_4x4mm_P0.5mm_EP2.3x2.3mm_ThermalVias" H 6675 4375 50  0001 C CNN
 F 3 "https://www.analog.com/media/en/technical-documentation/data-sheets/ADP5587.pdf" H 6675 4375 50  0001 C CNN
 F 4 "~" H 6275 3775 50  0001 C CNN "LcscNo"
