File: SequencerMidiController/PMOSReversePolarityProtection.kicad_sch (KiCad schematic)
At the start: 6 parts, among them Q1 Si2323DS

Commit message: Checked microSD card connector pins and added board layout connector footprint
Parts:
- D1: footprint Diode_SMD:D_SOD-123 -> Diode_SMD:D_SOD-123F
Changed lines of the file:
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@@
       (effects (font (size 1.27 1.27)) (justify left))
     )
-    (property "Footprint" "Diode_SMD:D_SOD-123" (id 2) (at 157.48 108.585 0)
+    (property "Footprint" "Diode_SMD:D_SOD-123F" (id 2) (at 157.48 108.585 0)
       (effects (font (size 1.27 1.27)) hide)
     )
